File: panel_v1/panel_v1.kicad_sch (KiCad schematic)
At the start: 0 parts

Commit message: starting work on monochrome screen
Parts:
- added J1: Conn_01x20, Connector_PinHeader_2.54mm:PinHeader_1x20_P2.54mm_Vertical, symbol Connector_Generic:Conn_01x20
Connections:
- new net GND: J1.1 (Pin_1), J1.13 (Pin_13), J1.17 (Pin_17), J1.2 (Pin_2), J1.9 (Pin_9)
- new net P_LED: J1.18 (Pin_18), J1.19 (Pin_19), J1.20 (Pin_20), J1.3 (Pin_3), J1.4 (Pin_4), J1.5 (Pin_5)
- new net ledArray/AMBER: J1.6 (Pin_6)
- new net ledArray/BLANK: J1.12 (Pin_12)
- new net ledArray/LATCH: J1.11 (Pin_11)
- new net ledArray/ROWblank: J1.16 (Pin_16)
- new net ledArray/ROWdat: J1.14 (Pin_14)
- new net ledArray/ROWlatch: J1.15 (Pin_15)
- new net ledArray/SCLK: J1.10 (Pin_10)
- no-connect marks 0 -> 2
Other:
- added sheet ledArray (ledArray.kicad_sch)
