File: panel_v1/ledArray.kicad_sch (KiCad schematic)
At the start: 20 parts, among them Q1 AO3401A, Q10 AO3401A, Q11 AO3401A, Q12 AO3401A, Q13 AO3401A, Q14 AO3401A, Q15 AO3401A, Q16 AO3401A, Q2 AO3401A, Q3 AO3401A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

Commit message: blinkenlites
Parts:
- removed U1, U2: 74HC595, Package_SO:TSSOP-16_4.4x5mm_P0.65mm, symbol 74xx:74HC595
- added U1, U2: 74AHC595, Package_SO:SSOP-16_5.3x6.2mm_P0.65mm, symbol 74xx:74AHC595
Connections:
- net GND: now also U1.8 (GND)
- net P_LED: now also U1.10 (~SRCLR), U1.16 (VCC), U2.10 (~SRCLR), U2.16 (VCC)
- net ROWblank: now also U1.13 (~OE), U2.13 (~OE)
- net ROWdat: now also U1.14 (SER)
- net ROWlatch: now also U1.12 (RCLK), U2.12 (RCLK)
- net SCLK: now also U1.11 (SRCLK), U2.11 (SRCLK)
- net at Q14.1 (G): now also U2.5 (QF)
- net at Q10.1 (G): now also U2.1 (QB)
- net at Q9.1 (G): now also U2.15 (QA)
- net at Q11.1 (G): now also U2.2 (QC)
- net at Q12.1 (G): now also U2.3 (QD)
- net at Q13.1 (G): now also U2.4 (QE)
- net at Q15.1 (G): now also U2.6 (QG)
- net at Q16.1 (G): now also U2.7 (QH)
- net at Q8.1 (G): now also U1.7 (QH)
- net at Q1.1 (G): now also U1.15 (QA)
- net at Q2.1 (G): now also U1.1 (QB)
- net at Q6.1 (G): now also U1.5 (QF)
- net at Q3.1 (G): now also U1.2 (QC)
- net at Q4.1 (G): now also U1.3 (QD)
- net at Q5.1 (G): now also U1.4 (QE)
- net at Q7.1 (G): now also U1.6 (QG)
- new net: U1.9 (QH'), U2.14 (SER)
Changed lines of the file:
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@@
-(kicad_sch (version 20200608) (host eeschema "5.99.0-unknown-e164269~101~ubuntu20.04.1")
+(kicad_sch (version 20200608) (host eeschema "5.99.0-unknown-0bfe413~101~ubuntu20.04.1")
   (page 2 19)
   (paper "A4")
@@
     )
   )
-  (symbol (lib_id "74xx:74HC595") (at 50.8 53.34 90) (mirror x) (unit 1)
-    (in_bom yes) (on_board yes)
-    (property "Reference" "U1" (id 0) (at 63.5 72.39 90)
+  (symbol (lib_id "74xx:74AHC595") (at 50.8 53.34 90) (mirror x) (unit 1)
+    (in_bom yes) (on_board yes)
+    (property "Reference" "U1" (id 0) (at 60.96 68.58 90)
       (effects (font (size 1.27 1.27)) (justify right))
     )
-    (property "Value" "74HC595" (id 1) (at 63.5 69.85 90)
+    (property "Value" "74AHC595" (id 1) (at 60.96 66.04 90)
       (effects (font (size 1.27 1.27)) (justify right))
     )
-    (property "Footprint" "Package_SO:TSSOP-16_4.4x5mm_P0.65mm" (id 2) (at 50.8 53.34 0)
-      (effects (font (size 1.27 1.27)) hide)
-    )
-    (property "Datasheet" "http://www.ti.com/lit/ds/symlink/sn74hc595.pdf" (id 3) (at 50.8 53.34 0)
-      (effects (font (size 1.27 1.27)) hide)
-    )
-  )
-  (symbol (lib_id "74xx:74HC595") (at 143.51 53.34 90) (mirror x) (unit 1)
-    (in_bom yes) (on_board yes)
-    (property "Reference" "U2" (id 0) (at 156.21 72.39 90)
+    (property "Footprint" "Package_SO:SSOP-16_5.3x6.2mm_P0.65mm" (id 2) (at 50.8 53.34 0)
+      (effects (font (size 1.27 1.27)) hide)
+    )
+    (property "Datasheet" "https://assets.nexperia.com/documents/data-sheet/74AHC_AHCT595.pdf" (id 3) (at 50.8 53.34 0)
+      (effects (font (size 1.27 1.27)) hide)
+    )
+  )
+  (symbol (lib_id "74xx:74AHC595") (at 143.51 53.34 90) (mirror x) (unit 1)
+    (in_bom yes) (on_board yes)
+    (property "Reference" "U2" (id 0) (at 153.67 68.58 90)
       (effects (font (size 1.27 1.27)) (justify right))
     )
-    (property "Value" "74HC595" (id 1) (at 156.21 69.85 90)
+    (property "Value" "74AHC595" (id 1) (at 153.67 66.04 90)
       (effects (font (size 1.27 1.27)) (justify right))
     )
-    (property "Footprint" "Package_SO:TSSOP-16_4.4x5mm_P0.65mm" (id 2) (at 143.51 53.34 0)
-      (effects (font (size 1.27 1.27)) hide)
-    )
-    (property "Datasheet" "http://www.ti.com/lit/ds/symlink/sn74hc595.pdf" (id 3) (at 143.51 53.34 0)
-      (effects (font (size 1.27 1.27)) hide)
-    )
+    (property "Footprint" "Package_SO:SSOP-16_5.3x6.2mm_P0.65mm" (id 2) (at 143.51 53.34 0)
+      (effects (font (size 1.27 1.27)) hide)
+    )
+    (property "Datasheet" "https://assets.nexperia.com/documents/data-sheet/74AHC_AHCT595.pdf" (id 3) (at 143.51 53.34 0)
+      (effects (font (size 1.27 1.27)) hide)
+    )
