File: panel_v1/ledStripe.kicad_sch (KiCad schematic)
At the start: 16 parts

Commit message: blinkenlites
Parts:
- renumbered D1 to D241, D2 to D242, D3 to D243, D4 to D244, D5 to D245, D6 to D246, D7 to D247, D8 to D248, D9 to D249, D10 to D250, D11 to D251, D12 to D252, D13 to D253, D14 to D254, D15 to D255, D16 to D256
Changed lines of the file:
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@@
-(kicad_sch (version 20200608) (host eeschema "5.99.0-unknown-e164269~101~ubuntu20.04.1")
-  (page 4 19)
+(kicad_sch (version 20200608) (host eeschema "5.99.0-unknown-0bfe413~101~ubuntu20.04.1")
+  (page 1 19)
   (paper "A4")
   (junction (at 82.55 57.15))
@@
   (symbol (lib_id "Device:LED") (at 82.55 50.8 270)
     (in_bom yes) (on_board yes)
-    (property "Reference" "D1" (id 0) (at 85.09 48.26 90)
+    (property "Reference" "D241" (id 0) (at 85.09 48.26 90)
       (effects (font (size 1.27 1.27)) (justify left))
     )
@@
   (symbol (lib_id "Device:LED") (at 91.44 50.8 270)
     (in_bom yes) (on_board yes)
-    (property "Reference" "D2" (id 0) (at 93.98 48.26 90)
+    (property "Reference" "D242" (id 0) (at 93.98 48.26 90)
       (effects (font (size 1.27 1.27)) (justify left))
     )
@@
   (symbol (lib_id "Device:LED") (at 100.33 50.8 270)
     (in_bom yes) (on_board yes)
-    (property "Reference" "D3" (id 0) (at 102.87 48.26 90)
+    (property "Reference" "D243" (id 0) (at 102.87 48.26 90)
       (effects (font (size 1.27 1.27)) (justify left))
     )
@@
   (symbol (lib_id "Device:LED") (at 109.22 50.8 270)
     (in_bom yes) (on_board yes)
-    (property "Reference" "D4" (id 0) (at 111.76 48.26 90)
+    (property "Reference" "D244" (id 0) (at 111.76 48.26 90)
       (effects (font (size 1.27 1.27)) (justify left))
     )
@@
   (symbol (lib_id "Device:LED") (at 118.11 50.8 270)
     (in_bom yes) (on_board yes)
-    (property "Reference" "D5" (id 0) (at 120.65 48.26 90)
+    (property "Reference" "D245" (id 0) (at 120.65 48.26 90)
       (effects (font (size 1.27 1.27)) (justify left))
     )
@@
   (symbol (lib_id "Device:LED") (at 127 50.8 270)
     (in_bom yes) (on_board yes)
-    (property "Reference" "D6" (id 0) (at 129.54 48.26 90)
+    (property "Reference" "D246" (id 0) (at 129.54 48.26 90)
       (effects (font (size 1.27 1.27)) (justify left))
     )
@@
   (symbol (lib_id "Device:LED") (at 135.89 50.8 270)
     (in_bom yes) (on_board yes)
-    (property "Reference" "D7" (id 0) (at 138.43 48.26 90)
+    (property "Reference" "D247" (id 0) (at 138.43 48.26 90)
       (effects (font (size 1.27 1.27)) (justify left))
     )
@@
   (symbol (lib_id "Device:LED") (at 144.78 50.8 270)
     (in_bom yes) (on_board yes)
-    (property "Reference" "D8" (id 0) (at 147.32 48.26 90)
+    (property "Reference" "D248" (id 0) (at 147.32 48.26 90)
       (effects (font (size 1.27 1.27)) (justify left))
     )
@@
   (symbol (lib_id "Device:LED") (at 154.94 50.8 270)
     (in_bom yes) (on_board yes)
-    (property "Reference" "D9" (id 0) (at 157.48 48.26 90)
+    (property "Reference" "D249" (id 0) (at 157.48 48.26 90)
       (effects (font (size 1.27 1.27)) (justify left))
     )
@@
   (symbol (lib_id "Device:LED") (at 163.83 50.8 270)
     (in_bom yes) (on_board yes)
-    (property "Reference" "D10" (id 0) (at 166.37 48.26 90)
+    (property "Reference" "D250" (id 0) (at 166.37 48.26 90)
       (effects (font (size 1.27 1.27)) (justify left))
     )
@@
   (symbol (lib_id "Device:LED") (at 172.72 50.8 270)
     (in_bom yes) (on_board yes)
-    (property "Reference" "D11" (id 0) (at 175.26 48.26 90)
+    (property "Reference" "D251" (id 0) (at 175.26 48.26 90)
       (effects (font (size 1.27 1.27)) (justify left))
     )
@@
   (symbol (lib_id "Device:LED") (at 181.61 50.8 270)
     (in_bom yes) (on_board yes)
-    (property "Reference" "D12" (id 0) (at 184.15 48.26 90)
+    (property "Reference" "D252" (id 0) (at 184.15 48.26 90)
       (effects (font (size 1.27 1.27)) (justify left))
     )
@@
   (symbol (lib_id "Device:LED") (at 190.5 50.8 270)
     (in_bom yes) (on_board yes)
-    (property "Reference" "D13" (id 0) (at 193.04 48.26 90)
+    (property "Reference" "D253" (id 0) (at 193.04 48.26 90)
       (effects (font (size 1.27 1.27)) (justify left))
     )
@@
   (symbol (lib_id "Device:LED") (at 199.39 50.8 270)
     (in_bom yes) (on_board yes)
-    (property "Reference" "D14" (id 0) (at 201.93 48.26 90)
+    (property "Reference" "D254" (id 0) (at 201.93 48.26 90)
       (effects (font (size 1.27 1.27)) (justify left))
     )
@@
   (symbol (lib_id "Device:LED") (at 208.28 50.8 270)
     (in_bom yes) (on_board yes)
-    (property "Reference" "D15" (id 0) (at 210.82 48.26 90)
+    (property "Reference" "D255" (id 0) (at 210.82 48.26 90)
       (effects (font (size 1.27 1.27)) (justify left))
     )
@@
   (symbol (lib_id "Device:LED") (at 217.17 50.8 270)
     (in_bom yes) (on_board yes)
-    (property "Reference" "D16" (id 0) (at 219.71 48.26 90)
-      (effects (font (size 1.27 1.27)) (justify left))
-    )
+    (property "Reference" "D256" (id 0) (at 219.71 48.26 90)
+      (effects (font (size 1.27 1.27)) (justify left))
+    )
