File: panel_v1/panel_v1.kicad_pcb (KiCad board)
At the start: 2 copper layers, 280 parts, among them J1 Conn_01x20, Q1 AO3401A, Q10 AO3401A, Q11 AO3401A, Q12 AO3401A, Q13 AO3401A, Q14 AO3401A, Q15 AO3401A, Q16 AO3401A, Q2 AO3401A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

Commit message: blinkenlites
Parts:
- moved D192 185.2 mm to (175.0, 155.0), turned to 30 degrees
- moved D242 184.8 mm to (105.0, 175.0), turned to 30 degrees
- moved D241 182.5 mm to (100.0, 175.0), turned to 30 degrees
- moved D191 179.6 mm to (170.0, 155.0), turned to 30 degrees
- moved D245 178.7 mm to (120.0, 175.0), turned to 30 degrees
- moved D244 176.3 mm to (115.0, 175.0), turned to 30 degrees
- moved D224 176.1 mm to (175.0, 165.0), turned to 30 degrees
- moved D246 173.6 mm to (125.0, 175.0), turned to 30 degrees
- moved D248 171.5 mm to (135.0, 175.0), turned to 30 degrees
- moved D189 170.9 mm to (160.0, 155.0), turned to 30 degrees
- moved D187 170.7 mm to (150.0, 155.0), turned to 30 degrees
- moved D223 170.3 mm to (170.0, 165.0), turned to 30 degrees
- moved D243 169.1 mm to (110.0, 175.0), turned to 30 degrees
- moved D190 168.7 mm to (165.0, 155.0), turned to 30 degrees
- moved D226 167.7 mm to (105.0, 170.0), turned to 30 degrees
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Other:
- board outline added: 66.8 x 67.8 mm
- net class Default removed
