File: rgb16/rgb16.kicad_sch (KiCad schematic)
At the start: 0 parts

Commit message: blinkenlites
Parts:
- added U? (x2): 74AHC595, symbol 74xx:74AHC595
- added U?: TLC5954, symbol JBC_TI:TLC5954
Changed lines of the file:
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@@
-(kicad_sch (version 20200310) (host eeschema "unknown")
-(  page "A4")
-  (symbol_instances)
+(kicad_sch (version 20200608) (host eeschema "5.99.0-unknown-0bfe413~101~ubuntu20.04.1")
+  (page 1 1)
+  (paper "A4")
+  (symbol (lib_id "74xx:74AHC595") (at 55.88 33.02 0) (unit 1)
+    (in_bom yes) (on_board yes)
+    (property "Reference" "U?" (id 0) (at 55.88 13.3158 0))
+    (property "Value" "74AHC595" (id 1) (at 55.88 15.6145 0))
+    (property "Footprint" "" (id 2) (at 55.88 33.02 0)
+      (effects (font (size 1.27 1.27)) hide)
+    )
+    (property "Datasheet" "https://assets.nexperia.com/documents/data-sheet/74AHC_AHCT595.pdf" (id 3) (at 55.88 33.02 0)
+      (effects (font (size 1.27 1.27)) hide)
+    )
+  )
+  (symbol (lib_id "74xx:74AHC595") (at 55.88 73.66 0) (unit 1)
+    (in_bom yes) (on_board yes)
+    (property "Reference" "U?" (id 0) (at 55.88 53.9558 0))
+    (property "Value" "74AHC595" (id 1) (at 55.88 56.2545 0))
+    (property "Footprint" "" (id 2) (at 55.88 73.66 0)
+      (effects (font (size 1.27 1.27)) hide)
+    )
+    (property "Datasheet" "https://assets.nexperia.com/documents/data-sheet/74AHC_AHCT595.pdf" (id 3) (at 55.88 73.66 0)
+      (effects (font (size 1.27 1.27)) hide)
+    )
+  )
+  (symbol (lib_id "JBC_TI:TLC5954") (at 140.97 107.95 0) (unit 1)
+    (in_bom yes) (on_board yes)
+    (property "Reference" "U?" (id 0) (at 139.065 117.3548 0))
+    (property "Value" "TLC5954" (id 1) (at 139.065 119.6535 0))
+    (property "Footprint" "" (id 2) (at 140.97 107.95 0)
+      (effects (font (size 1.27 1.27)) hide)
+    )
+    (property "Datasheet" "" (id 3) (at 140.97 107.95 0)
+      (effects (font (size 1.27 1.27)) hide)
+    )
+  )
+  (symbol_instances
+    (path "/3f817474-a524-4679-bd5c-ac5dbc3ee439"
+      (reference "U?") (unit 1)
+    )
+    (path "/72013e22-d8d2-4a3f-87ff-92e7b18049c1"
+      (reference "U?") (unit 1)
+    )
+    (path "/a25e440b-1f5a-4263-bf49-a3eb2f52435d"
+      (reference "U?") (unit 1)
+    )
+  )
 )
